File: PROBE-BOARD/PROBE-BOARD.kicad_pcb (KiCad board)
At the start: 2 copper layers, 15 x 31.7 mm, 9 parts, among them J1 Conn_01x01, J2 Conn_01x01, SW1 SW_Push_Open

Commit message: addd CADs and images
Other:
- board text added: "git.io/JkzZL"
Changed lines of the file:
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@@
   (general
     (thickness 1.6)
-    (drawings 30)
+    (drawings 32)
     (tracks 58)
     (zones 0)
@@
       (effects (font (size 1 1) (thickness 0.15)))
     )
+    (fp_circle (center 0 0) (end 3.2 0) (layer Cmts.User) (width 0.15))
     (fp_circle (center 0 0) (end 3.45 0) (layer F.CrtYd) (width 0.05))
-    (fp_circle (center 0 0) (end 3.2 0) (layer Cmts.User) (width 0.15))
     (fp_text user %R (at 0.3 0) (layer F.Fab)
       (effects (font (size 1 1) (thickness 0.15)))
@@
       (effects (font (size 1 1) (thickness 0.15)))
     )
+    (fp_circle (center 0 0) (end 3.2 0) (layer Cmts.User) (width 0.15))
     (fp_circle (center 0 0) (end 3.45 0) (layer F.CrtYd) (width 0.05))
-    (fp_circle (center 0 0) (end 3.2 0) (layer Cmts.User) (width 0.15))
     (fp_text user %R (at 0.3 0) (layer F.Fab)
       (effects (font (size 1 1) (thickness 0.15)))
@@
       (effects (font (size 1 1) (thickness 0.15)))
     )
+    (fp_line (start -6.35 -2.94) (end -6.35 2.94) (layer F.SilkS) (width 0.12))
+    (fp_line (start -6.35 2.94) (end 6.35 2.94) (layer F.SilkS) (width 0.12))
+    (fp_line (start 6.35 2.94) (end 6.35 -2.94) (layer F.SilkS) (width 0.12))
     (fp_line (start 6.35 -2.94) (end -6.35 -2.94) (layer F.SilkS) (width 0.12))
-    (fp_line (start 6.35 2.94) (end 6.35 -2.94) (layer F.SilkS) (width 0.12))
-    (fp_line (start -6.35 2.94) (end 6.35 2.94) (layer F.SilkS) (width 0.12))
-    (fp_line (start -6.35 -2.94) (end -6.35 2.94) (layer F.SilkS) (width 0.12))
     (pad 4 thru_hole circle (at 2.54 0 270) (size 1.6 1.6) (drill 0.8) (layers *.Cu *.Mask)
       (net 3 SIGNAL))
@@
       (effects (font (size 1 1) (thickness 0.15)) (justify mirror))
     )
+    (fp_line (start 1.65 -0.73) (end -1.65 -0.73) (layer B.CrtYd) (width 0.05))
+    (fp_line (start 1.65 0.73) (end 1.65 -0.73) (layer B.CrtYd) (width 0.05))
+    (fp_line (start -1.65 0.73) (end 1.65 0.73) (layer B.CrtYd) (width 0.05))
+    (fp_line (start -1.65 -0.73) (end -1.65 0.73) (layer B.CrtYd) (width 0.05))
+    (fp_line (start -0.254724 -0.5225) (end 0.254724 -0.5225) (layer B.SilkS) (width 0.12))
+    (fp_line (start -0.254724 0.5225) (end 0.254724 0.5225) (layer B.SilkS) (width 0.12))
+    (fp_line (start 0.8 -0.4125) (end -0.8 -0.4125) (layer B.Fab) (width 0.1))
+    (fp_line (start 0.8 0.4125) (end 0.8 -0.4125) (layer B.Fab) (width 0.1))
+    (fp_line (start -0.8 0.4125) (end 0.8 0.4125) (layer B.Fab) (width 0.1))
     (fp_line (start -0.8 -0.4125) (end -0.8 0.4125) (layer B.Fab) (width 0.1))
-    (fp_line (start -0.8 0.4125) (end 0.8 0.4125) (layer B.Fab) (width 0.1))
-    (fp_line (start 0.8 0.4125) (end 0.8 -0.4125) (layer B.Fab) (width 0.1))
-    (fp_line (start 0.8 -0.4125) (end -0.8 -0.4125) (layer B.Fab) (width 0.1))
-    (fp_line (start -0.254724 0.5225) (end 0.254724 0.5225) (layer B.SilkS) (width 0.12))
-    (fp_line (start -0.254724 -0.5225) (end 0.254724 -0.5225) (layer B.SilkS) (width 0.12))
-    (fp_line (start -1.65 -0.73) (end -1.65 0.73) (layer B.CrtYd) (width 0.05))
-    (fp_line (start -1.65 0.73) (end 1.65 0.73) (layer B.CrtYd) (width 0.05))
-    (fp_line (start 1.65 0.73) (end 1.65 -0.73) (layer B.CrtYd) (width 0.05))
-    (fp_line (start 1.65 -0.73) (end -1.65 -0.73) (layer B.CrtYd) (width 0.05))
     (fp_text user %R (at 0 0) (layer B.Fab)
       (effects (font (size 0.4 0.4) (thickness 0.06)) (justify mirror))
@@
       (effects (font (size 1 1) (thickness 0.15)))
     )
+    (fp_line (start 1.65 0.73) (end -1.65 0.73) (layer F.CrtYd) (width 0.05))
+    (fp_line (start 1.65 -0.73) (end 1.65 0.73) (layer F.CrtYd) (width 0.05))
+    (fp_line (start -1.65 -0.73) (end 1.65 -0.73) (layer F.CrtYd) (width 0.05))
+    (fp_line (start -1.65 0.73) (end -1.65 -0.73) (layer F.CrtYd) (width 0.05))
+    (fp_line (start -0.254724 0.5225) (end 0.254724 0.5225) (layer F.SilkS) (width 0.12))
+    (fp_line (start -0.254724 -0.5225) (end 0.254724 -0.5225) (layer F.SilkS) (width 0.12))
+    (fp_line (start 0.8 0.4125) (end -0.8 0.4125) (layer F.Fab) (width 0.1))
+    (fp_line (start 0.8 -0.4125) (end 0.8 0.4125) (layer F.Fab) (width 0.1))
+    (fp_line (start -0.8 -0.4125) (end 0.8 -0.4125) (layer F.Fab) (width 0.1))
     (fp_line (start -0.8 0.4125) (end -0.8 -0.4125) (layer F.Fab) (width 0.1))
-    (fp_line (start -0.8 -0.4125) (end 0.8 -0.4125) (layer F.Fab) (width 0.1))
-    (fp_line (start 0.8 -0.4125) (end 0.8 0.4125) (layer F.Fab) (width 0.1))
-    (fp_line (start 0.8 0.4125) (end -0.8 0.4125) (layer F.Fab) (width 0.1))
-    (fp_line (start -0.254724 -0.5225) (end 0.254724 -0.5225) (layer F.SilkS) (width 0.12))
-    (fp_line (start -0.254724 0.5225) (end 0.254724 0.5225) (layer F.SilkS) (width 0.12))
-    (fp_line (start -1.65 0.73) (end -1.65 -0.73) (layer F.CrtYd) (width 0.05))
-    (fp_line (start -1.65 -0.73) (end 1.65 -0.73) (layer F.CrtYd) (width 0.05))
-    (fp_line (start 1.65 -0.73) (end 1.65 0.73) (layer F.CrtYd) (width 0.05))
-    (fp_line (start 1.65 0.73) (end -1.65 0.73) (layer F.CrtYd) (width 0.05))
     (fp_text user %R (at 0 0) (layer F.Fab)
       (effects (font (size 0.4 0.4) (thickness 0.06)))
@@
   (module mag-probe:MagPad (layer F.Cu)
     (at 0 -10.75)
-    (fp_text reference J1 (at 3.556 3.638) (layer F.SilkS)
+    (fp_text reference J1 (at -3.7465 3.5745) (layer F.SilkS)
       (effects (font (size 1 1) (thickness 0.15)))
     )
@@
       (effects (font (size 1 1) (thickness 0.15)) (justify mirror))
     )
+    (fp_line (start 1.85 -0.95) (end -1.85 -0.95) (layer B.CrtYd) (width 0.05))
+    (fp_line (start 1.85 0.95) (end 1.85 -0.95) (layer B.CrtYd) (width 0.05))
+    (fp_line (start -1.85 0.95) (end 1.85 0.95) (layer B.CrtYd) (width 0.05))
+    (fp_line (start -1.85 -0.95) (end -1.85 0.95) (layer B.CrtYd) (width 0.05))
+    (fp_line (start -1.86 -0.96) (end 1 -0.96) (layer B.SilkS) (width 0.12))
+    (fp_line (start -1.86 0.96) (end -1.86 -0.96) (layer B.SilkS) (width 0.12))
+    (fp_line (start 1 0.96) (end -1.86 0.96) (layer B.SilkS) (width 0.12))
+    (fp_line (start 1 -0.6) (end 1 0.6) (layer B.Fab) (width 0.1))
+    (fp_line (start -1 -0.6) (end 1 -0.6) (layer B.Fab) (width 0.1))
+    (fp_line (start -1 0.3) (end -1 -0.6) (layer B.Fab) (width 0.1))
+    (fp_line (start -0.7 0.6) (end -1 0.3) (layer B.Fab) (width 0.1))
     (fp_line (start 1 0.6) (end -0.7 0.6) (layer B.Fab) (width 0.1))
-    (fp_line (start -0.7 0.6) (end -1 0.3) (layer B.Fab) (width 0.1))
-    (fp_line (start -1 0.3) (end -1 -0.6) (layer B.Fab) (width 0.1))
-    (fp_line (start -1 -0.6) (end 1 -0.6) (layer B.Fab) (width 0.1))
-    (fp_line (start 1 -0.6) (end 1 0.6) (layer B.Fab) (width 0.1))
-    (fp_line (start 1 0.96) (end -1.86 0.96) (layer B.SilkS) (width 0.12))
-    (fp_line (start -1.86 0.96) (end -1.86 -0.96) (layer B.SilkS) (width 0.12))
-    (fp_line (start -1.86 -0.96) (end 1 -0.96) (layer B.SilkS) (width 0.12))
-    (fp_line (start -1.85 -0.95) (end -1.85 0.95) (layer B.CrtYd) (width 0.05))
-    (fp_line (start -1.85 0.95) (end 1.85 0.95) (layer B.CrtYd) (width 0.05))
-    (fp_line (start 1.85 0.95) (end 1.85 -0.95) (layer B.CrtYd) (width 0.05))
-    (fp_line (start 1.85 -0.95) (end -1.85 -0.95) (layer B.CrtYd) (width 0.05))
     (fp_text user %R (at 0 0) (layer B.Fab)
       (effects (font (size 0.5 0.5) (thickness 0.08)) (justify mirror))
@@
       (effects (font (size 1 1) (thickness 0.15)))
     )
+    (fp_line (start 1.85 0.95) (end -1.85 0.95) (layer F.CrtYd) (width 0.05))
+    (fp_line (start 1.85 -0.95) (end 1.85 0.95) (layer F.CrtYd) (width 0.05))
+    (fp_line (start -1.85 -0.95) (end 1.85 -0.95) (layer F.CrtYd) (width 0.05))
+    (fp_line (start -1.85 0.95) (end -1.85 -0.95) (layer F.CrtYd) (width 0.05))
+    (fp_line (start -1.86 0.96) (end 1 0.96) (layer F.SilkS) (width 0.12))
+    (fp_line (start -1.86 -0.96) (end -1.86 0.96) (layer F.SilkS) (width 0.12))
+    (fp_line (start 1 -0.96) (end -1.86 -0.96) (layer F.SilkS) (width 0.12))
+    (fp_line (start 1 0.6) (end 1 -0.6) (layer F.Fab) (width 0.1))
+    (fp_line (start -1 0.6) (end 1 0.6) (layer F.Fab) (width 0.1))
+    (fp_line (start -1 -0.3) (end -1 0.6) (layer F.Fab) (width 0.1))
+    (fp_line (start -0.7 -0.6) (end -1 -0.3) (layer F.Fab) (width 0.1))
     (fp_line (start 1 -0.6) (end -0.7 -0.6) (layer F.Fab) (width 0.1))
-    (fp_line (start -0.7 -0.6) (end -1 -0.3) (layer F.Fab) (width 0.1))
-    (fp_line (start -1 -0.3) (end -1 0.6) (layer F.Fab) (width 0.1))
-    (fp_line (start -1 0.6) (end 1 0.6) (layer F.Fab) (width 0.1))
-    (fp_line (start 1 0.6) (end 1 -0.6) (layer F.Fab) (width 0.1))
-    (fp_line (start 1 -0.96) (end -1.86 -0.96) (layer F.SilkS) (width 0.12))
-    (fp_line (start -1.86 -0.96) (end -1.86 0.96) (layer F.SilkS) (width 0.12))
-    (fp_line (start -1.86 0.96) (end 1 0.96) (layer F.SilkS) (width 0.12))
-    (fp_line (start -1.85 0.95) (end -1.85 -0.95) (layer F.CrtYd) (width 0.05))
-    (fp_line (start -1.85 -0.95) (end 1.85 -0.95) (layer F.CrtYd) (width 0.05))
-    (fp_line (start 1.85 -0.95) (end 1.85 0.95) (layer F.CrtYd) (width 0.05))
-    (fp_line (start 1.85 0.95) (end -1.85 0.95) (layer F.CrtYd) (width 0.05))
     (fp_text user %R (at 0 0) (layer F.Fab)
       (effects (font (size 0.5 0.5) (thickness 0.08)))
@@
     )
   )
+  (gr_text git.io/JkzZL (at 5.715 10.16 90) (layer F.SilkS)
+    (effects (font (size 1 1) (thickness 0.15)))
+  )
+  (gr_text git.io/JkzZL (at 5.5245 10.414 90) (layer B.SilkS)
+    (effects (font (size 1 1) (thickness 0.15)) (justify mirror))
+  )
   (gr_text 1k (at -4.572 -1.905) (layer B.SilkS)
     (effects (font (size 1 1) (thickness 0.15)) (justify mirror))
@@
     (effects (font (size 1 1) (thickness 0.15)) (justify mirror))
   )
-  (gr_text J1 (at 3.556 -7.112) (layer B.SilkS)
-    (effects (font (size 1 1) (thickness 0.15)) (justify mirror))
-  )
+  (gr_text J1 (at -3.8735 -7.239) (layer B.SilkS)
+    (effects (font (size 1 1) (thickness 0.15)) (justify mirror))
+  )
