File: PROBE-BOARD/025mag-PROBE-BOARD.kicad_pcb (KiCad board)
At the start: 2 copper layers, 15 x 29.6 mm, 12 parts, among them SW1 SW_Push_Open

Commit message: README UPDATED
Parts:
- renumbered MAG1 to SIG
