File: PROBE-BOARD/PROBE-BOARD.sch (KiCad schematic (older format))
At the start: 7 parts, among them J1 Conn_01x01, J2 Conn_01x01, SW1 SW_Push_Open

Commit message: move M3  mounting holes, recreted CAD, added gerbers
Parts:
- R1: footprint Resistor_SMD:R_0603_1608Metric_Pad0.98x0.95mm_HandSolder -> Resistor_SMD:R_1206_3216Metric_Pad1.30x1.75mm_HandSolder
Changed lines of the file:
@@
 F 0 "R1" V 3800 1650 50  0000 C CNN
 F 1 "1k" V 4050 1650 50  0000 C CNN
-F 2 "Resistor_SMD:R_0603_1608Metric_Pad0.98x0.95mm_HandSolder" V 3880 1650 50  0001 C CNN
+F 2 "Resistor_SMD:R_1206_3216Metric_Pad1.30x1.75mm_HandSolder" V 3880 1650 50  0001 C CNN
 F 3 "~" H 3950 1650 50  0001 C CNN
 	1    3950 1650

Commit message: bOARD rev2
Parts:
- D1, D2: footprint LED_SMD:LED_0805_2012Metric_Pad1.15x1.40mm_HandSolder -> mag-probe:LED_1206_3216Metric_Pad1.42x1.75mm_HandSolder
Changed lines of the file:
@@
 F 0 "D2" H 3650 2100 50  0000 C CNN
 F 1 "LED_Small" H 3650 1900 50  0000 C CNN
-F 2 "LED_SMD:LED_0805_2012Metric_Pad1.15x1.40mm_HandSolder" V 3650 2000 50  0001 C CNN
+F 2 "mag-probe:LED_1206_3216Metric_Pad1.42x1.75mm_HandSolder" V 3650 2000 50  0001 C CNN
 F 3 "~" V 3650 2000 50  0001 C CNN
 	1    3650 2000
@@
 F 0 "D1" H 3650 1750 50  0000 C CNN
 F 1 "LED_Small" H 3650 1550 50  0000 C CNN
-F 2 "LED_SMD:LED_0805_2012Metric_Pad1.15x1.40mm_HandSolder" V 3650 1650 50  0001 C CNN
+F 2 "mag-probe:LED_1206_3216Metric_Pad1.42x1.75mm_HandSolder" V 3650 1650 50  0001 C CNN
 F 3 "~" V 3650 1650 50  0001 C CNN
 	1    3650 1650

Commit message: Rev2a of vias
Changed lines of the file:
@@
 Text GLabel 3450 1500 1    50   Input ~ 0
 SIGNAL
-Text Notes 6350 3500 0    50   ~ 0
+Text Notes 1100 2450 0    50   ~ 0
 1 - STP/SIGNAL\n2 - Vcc  (+3.3v / +5V)\n3 - GND
 Connection ~ 2400 3650
